File: Hardware/Lipo-Charger (base)/Switch Lipo Charger.kicad_pcb (KiCad board)
At the start: 2 copper layers, 30.8 x 15 mm, 23 parts, among them J1 USB_C_Receptacle_USB2.0, Q1 Si2307, SW1 JS202011SCQN, U2 LTC4054ES5-4.2

Commit message: Update Mechanic and Hardware
Parts:
- J1: value USB_C_Receptacle_USB2.0 -> GT-USB-7010ASV; footprint Connector_USB:USB_C_Receptacle_GCT_USB4085 -> Connector_USB:USB_C_Receptacle_G-Switch_GT-USB-7010ASV
- moved J1 4.82 mm to (112.5, 102.3)
- moved R4 0.06 mm to (104.9, 105.1)
- moved R5 0.06 mm to (106.4, 105.1)
- moved D2 0.05 mm to (106.2, 108.6)
Routing:
- net Net-(J1-CC1): track 15.3 -> 12.6 mm, vias 1 -> 2
- net VBUS: track 20.0 -> 17.5 mm
- net USB_D-: track 13.9 -> 15.3 mm
- net Net-(J1-CC2): track 6.87 -> 6.02 mm
- net USB_D+: track 13.8 -> 14.5 mm
Other:
- board text added: "LiPo Charger 2023-05-05"
- board text removed: "LiPo Charger 2023-03-25"
