File: Hardware/Lipo-Charger (base)/Switch Lipo Charger.kicad_sch (KiCad schematic)
At the start: 22 parts, among them J1 USB_C_Receptacle_USB2.0, Q1 Si2307, SW1 JS202011SCQN, U2 LTC4054ES5-4.2

Commit message: Update Mechanic and Hardware
Parts:
- J1: value USB_C_Receptacle_USB2.0 -> GT-USB-7010ASV; footprint Connector_USB:USB_C_Receptacle_GCT_USB4085 -> Connector_USB:USB_C_Receptacle_G-Switch_GT-USB-7010ASV
Changed lines of the file:
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@@
       (effects (font (size 1.27 1.27)))
     )
-    (property "Value" "USB_C_Receptacle_USB2.0" (at 71.12 64.135 0)
+    (property "Value" "GT-USB-7010ASV" (at 71.12 64.135 0)
       (effects (font (size 1.27 1.27)))
     )
-    (property "Footprint" "Connector_USB:USB_C_Receptacle_GCT_USB4085" (at 74.93 84.455 0)
+    (property "Footprint" "Connector_USB:USB_C_Receptacle_G-Switch_GT-USB-7010ASV" (at 74.93 84.455 0)
       (effects (font (size 1.27 1.27)) hide)
     )
